Commit message: working demo

File: turtlebot3_gix_description/ros2_control/turtlebot3_gix_system.ros2_control.xacro (robot description, xacro)
@@ -87,5 +87,5 @@
         </command_interface>
         <state_interface name="position">
-          <param name="initial_value">0.0</param>
+          <param name="initial_value">1.5708</param>
         </state_interface>
         <state_interface name="velocity">

File: turtlebot3_gix_description/urdf/gix_custom_add-on.urdf.xacro (robot description, xacro)
@@ -7,42 +7,16 @@
 <robot xmlns:xacro="http://www.ros.org/wiki/xacro">
   <xacro:macro name="gix_body" params="prefix">
-    <xacro:property
-      name="meshes_file_direction"
-      value="package://turtlebot3_manipulation_description/meshes/open_manipulator_x"/>
-    <link name="${prefix}link1">
+    <link name="${prefix}box_body">
       <visual>
-        <origin xyz="0 0 0" rpy="0 0 0"/>
+        <origin xyz="-0.01 0 0.072" rpy="0 0 0"/>
         <geometry>
-          <mesh filename="${meshes_file_direction}/link1.stl" scale="0.001 0.001 0.001"/>
+          <box size="0.192 0.154 0.144"/>
         </geometry>
-        <material name="grey"/>
+        <material name="yellow"/>
       </visual>
       <collision>
-        <origin xyz="0 0 0" rpy="0 0 0"/>
+        <origin xyz="-0.01 0 0.072" rpy="0 0 0"/>
         <geometry>
-          <box size="0.05 0.05 0.05"/>
-        </geometry>
-      </collision>
-    </link>
-    <joint name="${prefix}gix" type="revolute">
-      <parent link="${prefix}link1"/>
-      <child link="${prefix}link2"/>
-      <origin xyz="0.012 0.0 0.017" rpy="0 0 0"/>
-      <axis xyz="0 0 1"/>
-      <limit velocity="4.8" effort="1" lower="${-pi*0.9}" upper="${pi*0.9}" />
-      <dynamics damping="0.1"/>
-    </joint>
-    <link name="${prefix}link2">
-      <visual>
-        <origin xyz="0 0 0.019" rpy="0 0 0"/>
-        <geometry>
-          <mesh filename="${meshes_file_direction}/link2.stl" scale="0.001 0.001 0.001"/>
-        </geometry>
-        <material name="grey"/>
-      </visual>
-      <collision>
-        <origin xyz="0 0 0.019" rpy="0 0 0"/>
-        <geometry>
-          <mesh filename="${meshes_file_direction}/link2.stl" scale="0.001 0.001 0.001"/>
+          <box size="192.0 154.0 144.0"/>
         </geometry>
       </collision>

File: turtlebot3_gix_description/urdf/materials.xacro (robot description, xacro)
@@ -35,3 +35,6 @@
     <color rgba="1.0 1.0 1.0 1.0"/>
   </material>
+  <material name="yellow">
+    <color rgba="1.0 1.0 0.0 1.0"/>
+  </material>
 </robot>

File: turtlebot3_gix_description/urdf/turtlebot3_burger.urdf.xacro (robot description, xacro)
@@ -15,5 +15,5 @@
       <origin xyz="-0.032 0 0.0" rpy="0 0 0"/>
       <geometry>
-        <mesh filename="${meshes_file_direction}/burger_base.stl" scale="0.001 0.001 0.001"/>
+        <mesh filename="${meshes_file_direction}/base.stl" scale="0.001 0.001 0.001"/>
       </geometry>
       <material name="light_black"/>

File: turtlebot3_gix_description/urdf/turtlebot3_gix.urdf.xacro (robot description, xacro)
@@ -15,9 +15,9 @@
   <xacro:include filename="$(find turtlebot3_gix_description)/ros2_control/turtlebot3_gix_system.ros2_control.xacro" />
   <xacro:turtlebot3_burger prefix="$(arg prefix)" />
-  <!-- Used for fixing OpenManipulator-X on TurtleBot3 Waffle Pi -->
+  <!-- Used for fixing custom additions to TurtleBot3 -->
   <joint name="$(arg prefix)base_fixed" type="fixed">
     <parent link="$(arg prefix)base_link"/>
-    <child link="$(arg prefix)link1"/>
-    <origin xyz="-0.092 0.0 0.091" rpy="0 0 0"/>
+    <child link="$(arg prefix)box_body"/>
+    <origin xyz="0.0 0.0 0.0" rpy="0 0 0"/>
   </joint>
   <xacro:gix_body prefix="$(arg prefix)" />
